File: kicad/pico-w-rotator/pico-w-rotator.kicad_sch (KiCad schematic)
At the start: 163 parts, among them J1 DB9_Male, SW1 Mode Button, U1 PicoW, U2 MAX3232, U3 LM7805_TO220

Commit message: config stuff.
Other:
- title: N1KDO Pico-W Rotator IOT Interface -> PICO-W Wireless Rotator Controller
Changed lines of the file:
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@@
   (paper "A")
   (title_block
-    (title "N1KDO Pico-W Rotator IOT Interface")
-    (date "2022-08-17")
-    (rev "0.1")
+    (title "PICO-W Wireless Rotator Controller")
+    (date "2022-08-21")
+    (rev "0.2")
+    (comment 4 "Copyright (C) 2022 J. B. Otterson N1KDO")
   )
   (junction (at 30.48 196.85) (diameter 0) (color 0 0 0 0)

Commit message: pcb measured, checked
sent out to oshpark!

schem changed, sanity
Parts:
- removed TP7: TestPoint, TestPoint:TestPoint_THTPad_D1.0mm_Drill0.5mm, symbol Connector:TestPoint
Changed lines of the file:
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@@
     )
-  )
-  (symbol (lib_id "Connector:TestPoint") (at 83.82 58.42 90) (unit 1)
-    (in_bom yes) (on_board yes)
-    (property "Reference" "TP7" (id 0) (at 77.47 58.42 90))
-    (property "Value" "TestPoint" (id 1) (at 80.518 56.6221 90)
-      (effects (font (size 1.27 1.27)) hide)
-    )
-    (property "Footprint" "TestPoint:TestPoint_THTPad_D1.0mm_Drill0.5mm" (id 2) (at 83.82 53.34 0)
-      (effects (font (size 1.27 1.27)) hide)
-    )
-    (property "Datasheet" "~" (id 3) (at 83.82 53.34 0)
-      (effects (font (size 1.27 1.27)) hide)
-    )
-    (pin "1")
   )
   (symbol (lib_id "Connector:TestPoint") (at 119.38 78.74 270) (unit 1)
@@
       (reference "TP6") (unit 1) (value "TestPoint") (footprint "TestPoint:TestPoint_THTPad_D1.0mm_Drill0.5mm")
     )
-    (path "/80fe2e45-744a-45a1-be79-ff4a1c6cb9ff"
-      (reference "TP7") (unit 1) (value "TestPoint") (footprint "TestPoint:TestPoint_THTPad_D1.0mm_Drill0.5mm")
-    )
     (path "/bbd15443-3b01-4f95-b94b-2795f7576bd6"
